Commit message: Support ros2_control.  moveit2 support next.

File: xarm_description/urdf/xarm.urdf (robot description, URDF)
Before this commit: robot xarm, 6 links, 5 joints
Links:
- link xarm_base_link: mass 0.1 -> None

Commit message: Add support for Gripper
Controllable using test_xarm_gripper_position_controller.launch.py. WIP
for moveit.

File: xarm_description/urdf/xarm.urdf (robot description, URDF)
Before this commit: robot xarm, 6 links, 5 joints
Links:
- added link xarm_gripper_base_link, mass 0.1; collision mesh filename=package://xarm_description/meshes/stls/gripper_palm.stl scale=1.0 1.0 1.0; visual mesh filename=package://xarm_description/meshes/stls/gripper_palm.stl scale=1.0 1.0 1.0
- added link xarm_gripper_finger_left_link, mass 0.1; collision mesh filename=package://xarm_description/meshes/stls/gripper_finger_left.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 scale=1.0 1.0 1.0; visual mesh filename=package://xarm_description/meshes/stls/gripper_finger_left.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 scale=1.0 1.0 1.0
- added link xarm_gripper_finger_right_link, mass 0.1; collision mesh filename=package://xarm_description/meshes/stls/gripper_finger_right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 scale=1.0 1.0 1.0; visual mesh filename=package://xarm_description/meshes/stls/gripper_finger_right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 scale=1.0 1.0 1.0
Joints:
- added joint xarm_1_joint: type prismatic, parent xarm_gripper_base_link, child xarm_gripper_finger_left_link, origin xyz=0 0 0.050 rpy=0 0 0, axis 1 0 0, limit lower=0.003 upper=0.028 effort=1000.0 velocity=0.5
- added joint xarm_1_joint_mirror: type prismatic, parent xarm_gripper_base_link, child xarm_gripper_finger_right_link, origin xyz=0 0 0.050 rpy=0 0 0, axis 1 0 0, limit lower=0.003 upper=0.028 effort=1000.0 velocity=0.5, mimic joint=xarm_1_joint multiplier=-1.0
- added joint xarm_end_effector_joint: type fixed, parent xarm_2_link, child xarm_gripper_base_link, origin xyz=0 0 0 rpy=0 0 0, axis 0 0 1

Commit message: Combine xarm_2_link with xarm_gripper_base_link so that an IkFast solver can be generated.  Other cleanup.

File: xarm_description/urdf/xarm.urdf (robot description, URDF)
Before this commit: robot xarm, 9 links, 8 joints
Links:
- removed link xarm_2_link
Joints:
- removed joint xarm_end_effector_joint
- joint xarm_2_joint: axis 0 0 1 -> 0 1 0; child xarm_2_link -> xarm_gripper_base_link

Commit message: Add support for revised xArm that has an additional joint for a total of 6DOF

File: xarm_description/urdf/xarm.urdf (robot description, URDF)
Before this commit: robot xarm, 8 links, 7 joints
Links:
- added link xarm_7_link, mass 0.1; collision mesh filename=package://xarm_description/meshes/stls/link2.stl scale=1.0 1.0 1.0; visual mesh filename=package://xarm_description/meshes/stls/link7_6dof.stl scale=1.0 1.0 1.0
- link xarm_4_link: geometry visual mesh filename=package://xarm_description/meshes/stls/link4_6dof.stl scale=1.0 1.0 1.0
Joints:
- added joint xarm_7_joint: type revolute, parent xarm_4_link, child xarm_7_link, origin xyz=0 0 0.090 rpy=0 0 0, axis 0 0 1, limit lower=-1.57 upper=1.57 effort=1000 velocity=1.0
- joint xarm_2_joint: axis 0 1 0 -> 0 0 1; limit lower=-2.17494876 upper=1.63121157 effort=1000 velocity=1.0 -> lower=-1.208 upper=1.933 effort=1000 velocity=1.0
- joint xarm_3_joint: origin xyz=0 0.0 0.09825 rpy=0 0 0 -> xyz=0 0.0 0.030 rpy=0 0 0; parent xarm_4_link -> xarm_7_link
- joint xarm_4_joint: origin xyz=0 0.0 0.09765 rpy=0 0 0 -> xyz=0 0.0 0.097 rpy=0 0 0

Commit message: Cleanup

File: xarm_description/urdf/xarm.urdf (robot description, URDF)
Before this commit: robot xarm, 9 links, 8 joints
Links:
- link xarm_4_link: geometry collision mesh filename=package://xarm_description/meshes/stls/link4_6dof.stl scale=1.0 1.0 1.0; visual mesh filename=package://xarm_description/meshes/stls/link4_6dof.stl scale=1.0 1.0 1.0
- link xarm_7_link: geometry collision mesh filename=package://xarm_description/meshes/stls/link7_6dof.stl scale=1.0 1.0 1.0; visual mesh filename=package://xarm_description/meshes/stls/link7_6dof.stl scale=1.0 1.0 1.0

Commit message: Add support for 3-finger end effector

File: xarm_description/urdf/xarm.urdf (robot description, URDF)
Before this commit: robot xarm, 9 links, 8 joints
Links:
- removed link xarm_gripper_base_link
- removed link xarm_gripper_finger_left_link
- removed link xarm_gripper_finger_right_link
Joints:
- removed joint xarm_1_joint
- removed joint xarm_1_joint_mirror
- joint xarm_2_joint: child xarm_gripper_base_link -> (none)

File: xarm_description/urdf/xarm_world.urdf.xacro (robot description, xacro)
@@ -1,3 +1,4 @@
 <robot xmlns:xacro="http://ros.org/wiki/xacro" name="xarm">
+    <xacro:property name="eef" value="eef_3_finger"/>
     <xacro:include filename="$(find xarm_description)/urdf/xarm.urdf"/>
     <link name="world"/>
